Commit message: megarover_samplesをmodelに統一

File: model/robots/megarover.urdf (robot description, URDF)
Before this commit: robot megarover20, 3 links, 2 joints
Links:
- link base_link: geometry visual mesh filename=/home/rover/catkin_ws/src/model/meshes/DAE/megarover.dae

File: model/robots/megarover.urdf.xacro (robot description, xacro)
@@ -1,5 +1,5 @@
 <?xml version="1.0"?>
 <robot name="megarover20" xmlns:xacro="http://ros.org/wiki/xacro">
-  <xacro:include filename="$(find megarover_samples)/urdf/body/body.urdf.xacro"/>
+  <xacro:include filename="$(find model)/urdf/body/body.urdf.xacro"/>
   <link name="base_footprint"/>
   <xacro:body parent="base_footprint">

File: model/robots/vmegarover.urdf.xacro (robot description, xacro)
@@ -1,7 +1,7 @@
 <?xml version="1.0"?>
 <robot name="vmegarover" xmlns:xacro="http://ros.org/wiki/xacro">
-  <xacro:include filename="$(find megarover_samples)/urdf/body/vbody.urdf.xacro"/>
-  <xacro:include filename="$(find megarover_samples)/urdf/wheel/vwheel.urdf.xacro"/>
-  <xacro:include filename="$(find megarover_samples)/urdf/lrf/lrf.urdf.xacro"/>
+  <xacro:include filename="$(find model)/urdf/body/vbody.urdf.xacro"/>
+  <xacro:include filename="$(find model)/urdf/wheel/vwheel.urdf.xacro"/>
+  <xacro:include filename="$(find model)/urdf/lrf/lrf.urdf.xacro"/>
   <!-- =============== Link & Joint =============== -->
   <!-- Base -->
